Commit message: cleanup

File: catkin_ws/src/my_robot/urdf/immovable.urdf (robot description, URDF)
Before this commit: robot xd, 5 links, 4 joints
Links:
- link link1: geometry visual box size=${params['s2']['link_l']} ${link_w} ${link_w}
- link link2: geometry visual box size=${params['s3']['link_l']} ${link_w} ${link_w}
Joints:
- joint joint1: origin xyz=0 0 0 rpy=0 0 0 -> xyz=${params['s1']['joint_xyz']} rpy=${params['s1']['joint_rpy']}; type continuous -> fixed
- joint joint2: origin xyz=0 0 0 rpy=-1.57 0 0 -> xyz=${params['s2']['joint_xyz']} rpy=${params['s2']['joint_rpy']}; type continuous -> fixed
- joint joint3: origin xyz=0.5 0 0 rpy=0 0 0 -> xyz=${params['s3']['joint_xyz']} rpy=${params['s3']['joint_rpy']}; type continuous -> fixed
